Commit message: urdf changes for simulation

File: acrux_description/urdf/acrux.xacro (robot description, xacro)
@@ -13,5 +13,5 @@
     <origin xyz="0 0 0" rpy="0 0 0"/>
     <geometry>
-      <mesh filename="package://acrux_description/meshes/base_link.dae" scale="0.001 0.001 0.001"/>
+      <mesh filename="file://$(find acrux_description)/meshes/base_link.dae" scale="0.001 0.001 0.001"/>
     </geometry>
     <material name="silver"/>
@@ -20,5 +20,5 @@
     <origin xyz="0 0 0" rpy="0 0 0"/>
     <geometry>
-      <mesh filename="package://acrux_description/meshes/base_link.dae" scale="0.001 0.001 0.001"/>
+      <mesh filename="file://$(find acrux_description)/meshes/base_link.dae" scale="0.001 0.001 0.001"/>
     </geometry>
   </collision>
@@ -33,5 +33,5 @@
     <origin xyz="-0.250058 0.175387 -0.06065" rpy="0 0 0"/>
     <geometry>
-      <mesh filename="package://acrux_description/meshes/rf_caster_holder_1.stl" scale="0.001 0.001 0.001"/>
+      <mesh filename="file://$(find acrux_description)/meshes/rf_caster_holder_1.stl" scale="0.001 0.001 0.001"/>
     </geometry>
     <material name="silver"/>
@@ -40,5 +40,5 @@
     <origin xyz="-0.250058 0.175387 -0.06065" rpy="0 0 0"/>
     <geometry>
-      <mesh filename="package://acrux_description/meshes/rf_caster_holder_1.stl" scale="0.001 0.001 0.001"/>
+      <mesh filename="file://$(find acrux_description)/meshes/rf_caster_holder_1.stl" scale="0.001 0.001 0.001"/>
     </geometry>
   </collision>
@@ -53,5 +53,5 @@
     <origin xyz="-0.22071 0.174967 -0.027246" rpy="0 0 0"/>
     <geometry>
-      <mesh filename="package://acrux_description/meshes/rf_caster_wheel_1.stl" scale="0.001 0.001 0.001"/>
+      <mesh filename="file://$(find acrux_description)/meshes/rf_caster_wheel_1.stl" scale="0.001 0.001 0.001"/>
     </geometry>
     <material name="silver"/>
@@ -60,5 +60,5 @@
     <origin xyz="-0.22071 0.174967 -0.027246" rpy="0 0 0"/>
     <geometry>
-      <mesh filename="package://acrux_description/meshes/rf_caster_wheel_1.stl" scale="0.001 0.001 0.001"/>
+      <mesh filename="file://$(find acrux_description)/meshes/rf_caster_wheel_1.stl" scale="0.001 0.001 0.001"/>
     </geometry>
   </collision>
@@ -73,5 +73,5 @@
     <origin xyz="-0.250058 -0.175387 -0.06065" rpy="0 0 0"/>
     <geometry>
-      <mesh filename="package://acrux_description/meshes/lf_caster_holder_1.stl" scale="0.001 0.001 0.001"/>
+      <mesh filename="file://$(find acrux_description)/meshes/lf_caster_holder_1.stl" scale="0.001 0.001 0.001"/>
     </geometry>
     <material name="silver"/>
@@ -80,5 +80,5 @@
     <origin xyz="-0.250058 -0.175387 -0.06065" rpy="0 0 0"/>
     <geometry>
-      <mesh filename="package://acrux_description/meshes/lf_caster_holder_1.stl" scale="0.001 0.001 0.001"/>
+      <mesh filename="file://$(find acrux_description)/meshes/lf_caster_holder_1.stl" scale="0.001 0.001 0.001"/>
     </geometry>
   </collision>
@@ -93,5 +93,5 @@
     <origin xyz="-0.22071 -0.174967 -0.024259" rpy="0 0 0"/>
     <geometry>
-      <mesh filename="package://acrux_description/meshes/lf_caster_wheel_1.stl" scale="0.001 0.001 0.001"/>
+      <mesh filename="file://$(find acrux_description)/meshes/lf_caster_wheel_1.stl" scale="0.001 0.001 0.001"/>
     </geometry>
     <material name="silver"/>
@@ -100,5 +100,5 @@
     <origin xyz="-0.22071 -0.174967 -0.024259" rpy="0 0 0"/>
     <geometry>
-      <mesh filename="package://acrux_description/meshes/lf_caster_wheel_1.stl" scale="0.001 0.001 0.001"/>
+      <mesh filename="file://$(find acrux_description)/meshes/lf_caster_wheel_1.stl" scale="0.001 0.001 0.001"/>
     </geometry>
   </collision>
@@ -113,5 +113,5 @@
     <origin xyz="-0.283 -0.0 -0.1599" rpy="0 0 0"/>
     <geometry>
-      <mesh filename="package://acrux_description/meshes/lidar_1.stl" scale="0.001 0.001 0.001"/>
+      <mesh filename="file://$(find acrux_description)/meshes/lidar_1.stl" scale="0.001 0.001 0.001"/>
     </geometry>
     <material name="silver"/>
@@ -120,5 +120,5 @@
     <origin xyz="-0.283 -0.0 -0.1599" rpy="0 0 0"/>
     <geometry>
-      <mesh filename="package://acrux_description/meshes/lidar_1.stl" scale="0.001 0.001 0.001"/>
+      <mesh filename="file://$(find acrux_description)/meshes/lidar_1.stl" scale="0.001 0.001 0.001"/>
     </geometry>
   </collision>
@@ -133,5 +133,5 @@
     <origin xyz="0.250058 -0.175566 -0.06065" rpy="0 0 0"/>
     <geometry>
-      <mesh filename="package://acrux_description/meshes/lb_caster_holder_1.stl" scale="0.001 0.001 0.001"/>
+      <mesh filename="file://$(find acrux_description)/meshes/lb_caster_holder_1.stl" scale="0.001 0.001 0.001"/>
     </geometry>
     <material name="silver"/>
@@ -140,5 +140,5 @@
     <origin xyz="0.250058 -0.175566 -0.06065" rpy="0 0 0"/>
     <geometry>
-      <mesh filename="package://acrux_description/meshes/lb_caster_holder_1.stl" scale="0.001 0.001 0.001"/>
+      <mesh filename="file://$(find acrux_description)/meshes/lb_caster_holder_1.stl" scale="0.001 0.001 0.001"/>
     </geometry>
   </collision>
@@ -153,5 +153,5 @@
     <origin xyz="0.22071 -0.175146 -0.024259" rpy="0 0 0"/>
     <geometry>
-      <mesh filename="package://acrux_description/meshes/lb_caster_wheel_1.stl" scale="0.001 0.001 0.001"/>
+      <mesh filename="file://$(find acrux_description)/meshes/lb_caster_wheel_1.stl" scale="0.001 0.001 0.001"/>
     </geometry>
     <material name="silver"/>
@@ -160,5 +160,5 @@
     <origin xyz="0.22071 -0.175146 -0.024259" rpy="0 0 0"/>
     <geometry>
-      <mesh filename="package://acrux_description/meshes/lb_caster_wheel_1.stl" scale="0.001 0.001 0.001"/>
+      <mesh filename="file://$(find acrux_description)/meshes/lb_caster_wheel_1.stl" scale="0.001 0.001 0.001"/>
     </geometry>
   </collision>
@@ -173,5 +173,5 @@
     <origin xyz="0.000209 -0.232679 -0.06" rpy="0 0 0"/>
     <geometry>
-      <mesh filename="package://acrux_description/meshes/left_wheel_1.stl" scale="0.001 0.001 0.001"/>
+      <mesh filename="file://$(find acrux_description)/meshes/left_wheel_1.stl" scale="0.001 0.001 0.001"/>
     </geometry>
     <material name="silver"/>
@@ -180,5 +180,5 @@
     <origin xyz="0.000209 -0.232679 -0.06" rpy="0 0 0"/>
     <geometry>
-      <mesh filename="package://acrux_description/meshes/left_wheel_1.stl" scale="0.001 0.001 0.001"/>
+      <mesh filename="file://$(find acrux_description)/meshes/left_wheel_1.stl" scale="0.001 0.001 0.001"/>
     </geometry>
   </collision>
@@ -193,5 +193,5 @@
     <origin xyz="0.0 0.232322 -0.06" rpy="0 0 0"/>
     <geometry>
-      <mesh filename="package://acrux_description/meshes/right_wheel_1.stl" scale="0.001 0.001 0.001"/>
+      <mesh filename="file://$(find acrux_description)/meshes/right_wheel_1.stl" scale="0.001 0.001 0.001"/>
     </geometry>
     <material name="silver"/>
@@ -200,5 +200,5 @@
     <origin xyz="0.0 0.232322 -0.06" rpy="0 0 0"/>
     <geometry>
-      <mesh filename="package://acrux_description/meshes/right_wheel_1.stl" scale="0.001 0.001 0.001"/>
+      <mesh filename="file://$(find acrux_description)/meshes/right_wheel_1.stl" scale="0.001 0.001 0.001"/>
     </geometry>
   </collision>
@@ -213,5 +213,5 @@
     <origin xyz="0.250058 0.175209 -0.06065" rpy="0 0 0"/>
     <geometry>
-      <mesh filename="package://acrux_description/meshes/rb_caster_holder_1.stl" scale="0.001 0.001 0.001"/>
+      <mesh filename="file://$(find acrux_description)/meshes/rb_caster_holder_1.stl" scale="0.001 0.001 0.001"/>
     </geometry>
     <material name="silver"/>
@@ -220,5 +220,5 @@
     <origin xyz="0.250058 0.175209 -0.06065" rpy="0 0 0"/>
     <geometry>
-      <mesh filename="package://acrux_description/meshes/rb_caster_holder_1.stl" scale="0.001 0.001 0.001"/>
+      <mesh filename="file://$(find acrux_description)/meshes/rb_caster_holder_1.stl" scale="0.001 0.001 0.001"/>
     </geometry>
   </collision>
@@ -233,5 +233,5 @@
     <origin xyz="0.22071 0.174789 -0.024259" rpy="0 0 0"/>
     <geometry>
-      <mesh filename="package://acrux_description/meshes/rb_caster_wheel_1.stl" scale="0.001 0.001 0.001"/>
+      <mesh filename="file://$(find acrux_description)/meshes/rb_caster_wheel_1.stl" scale="0.001 0.001 0.001"/>
     </geometry>
     <material name="silver"/>
@@ -240,5 +240,5 @@
     <origin xyz="0.22071 0.174789 -0.024259" rpy="0 0 0"/>
     <geometry>
-      <mesh filename="package://acrux_description/meshes/rb_caster_wheel_1.stl" scale="0.001 0.001 0.001"/>
+      <mesh filename="file://$(find acrux_description)/meshes/rb_caster_wheel_1.stl" scale="0.001 0.001 0.001"/>
     </geometry>
   </collision>
@@ -253,5 +253,5 @@
     <origin xyz="0.125 0.174821 -0.069" rpy="0 0 0"/>
     <geometry>
-      <mesh filename="package://acrux_description/meshes/right_suspension_1.stl" scale="0.001 0.001 0.001"/>
+      <mesh filename="file://$(find acrux_description)/meshes/right_suspension_1.stl" scale="0.001 0.001 0.001"/>
     </geometry>
     <material name="silver"/>
@@ -260,5 +260,5 @@
     <origin xyz="0.125 0.174821 -0.069" rpy="0 0 0"/>
     <geometry>
-      <mesh filename="package://acrux_description/meshes/right_suspension_1.stl" scale="0.001 0.001 0.001"/>
+      <mesh filename="file://$(find acrux_description)/meshes/right_suspension_1.stl" scale="0.001 0.001 0.001"/>
     </geometry>
   </collision>
@@ -273,5 +273,5 @@
     <origin xyz="0.125 -0.174822 -0.069" rpy="0 0 0"/>
     <geometry>
-      <mesh filename="package://acrux_description/meshes/left_suspension_1.stl" scale="0.001 0.001 0.001"/>
+      <mesh filename="file://$(find acrux_description)/meshes/left_suspension_1.stl" scale="0.001 0.001 0.001"/>
     </geometry>
     <material name="silver"/>
@@ -280,5 +280,5 @@
     <origin xyz="0.125 -0.174822 -0.069" rpy="0 0 0"/>
     <geometry>
-      <mesh filename="package://acrux_description/meshes/left_suspension_1.stl" scale="0.001 0.001 0.001"/>
+      <mesh filename="file://$(find acrux_description)/meshes/left_suspension_1.stl" scale="0.001 0.001 0.001"/>
     </geometry>
   </collision>
@@ -293,5 +293,5 @@
     <origin xyz="-0.318 0.0 -0.093001" rpy="0 0 0"/>
     <geometry>
-      <mesh filename="package://acrux_description/meshes/camera_link_1.dae" scale="0.001 0.001 0.001"/>
+      <mesh filename="file://$(find acrux_description)/meshes/camera_link_1.dae" scale="0.001 0.001 0.001"/>
     </geometry>
     <material name="silver"/>
@@ -300,5 +300,5 @@
     <origin xyz="-0.318 0.0 -0.093001" rpy="0 0 0"/>
     <geometry>
-      <mesh filename="package://acrux_description/meshes/camera_link_1.dae" scale="0.001 0.001 0.001"/>
+      <mesh filename="file://$(find acrux_description)/meshes/camera_link_1.dae" scale="0.001 0.001 0.001"/>
     </geometry>
   </collision>
